Commit message: manipulator example added

File: robot_model/manipulator/three_link_manipulator.urdf (robot description, URDF)
Before this commit: robot 2link_robot, 5 links, 4 joints
Links:
- removed link l0
- added link world, mass 1.
- link ee: geometry visual sphere radius=0.05
Joints:
- joint ee_joint: origin xyz=1 0 0 rpy=0 0 0 -> xyz=1.0 0 0 rpy=0 0 0
- joint j0: limit (none) -> lower=-6.28318530718 upper=6.28318530718 effort=150.0 velocity=3.15; parent l0 -> world; type continuous -> revolute
- joint j1: limit (none) -> lower=-6.28318530718 upper=6.28318530718 effort=150.0 velocity=3.15; type continuous -> revolute
- joint j2: limit (none) -> lower=-6.28318530718 upper=6.28318530718 effort=150.0 velocity=3.15; type continuous -> revolute
