Commit message: atlas balancing

File: robot_model/atlas/atlas.urdf (robot description, URDF)
Before this commit: robot multisense_sl, 33 links, 32 joints
Links:
- added link pelvis_com, mass 0.001
- link head: geometry collision box size=0.0468 0.12 0.1184; collision box size=0.1311 0.12 0.0591
- link l_clav: geometry collision box size=0.1 0.07 0.072; collision cylinder length=0.1525 radius=0.0555
- link l_foot: geometry collision box size=0.1 0.08 0.02; collision box size=0.227 0.133887 0.05
- link l_larm: geometry collision box size=0.135 0.15 0.06; collision cylinder length=0.125 radius=0.045
- link l_lfarm: geometry collision box size=0.13 0.09 0.07; collision cylinder length=0.05 radius=0.03
- link l_lglut: geometry collision box size=0.125 0.05 0.08; collision cylinder length=0.060306 radius=0.02009687
- link l_lleg: geometry collision cylinder length=0.40 radius=0.07; visual mesh filename=package://meshes_unplugged/l_lleg.obj scale=1 1 1
- link l_scap: geometry collision box size=0.02 0.029 0.018; collision box size=0.028 0.090 0.05
- link l_talus: geometry collision cylinder length=0.010059 radius=0.010348; collision cylinder length=0.029542 radius=0.010181
- link l_uarm: geometry collision box size=0.05 0.07 0.15; collision cylinder length=0.11 radius=0.065
- link l_ufarm: geometry collision box size=0.135 0.1 0.045; collision cylinder length=0.125 radius=0.045
- link l_uglut: geometry collision box size=0.05 0.1 0.1; collision cylinder length=0.080842 radius=0.019841
- link l_uleg: geometry collision box size=0.07 0.038 0.14; collision box size=0.07 0.038 0.15
- link ltorso: geometry visual mesh filename=package://meshes_unplugged/ltorso.obj scale=1 1 1
- link mtorso: geometry collision cylinder length=0.15 radius=0.02; visual mesh filename=package://meshes_unplugged/mtorso.obj scale=1 1 1
- link pelvis: geometry collision box size=0.1 0.15 0.2; collision cylinder length=0.05 radius=0.16
- link r_clav: geometry collision box size=0.1 0.07 0.072; collision cylinder length=0.1525 radius=0.0555
- link r_foot: geometry collision box size=0.1 0.08 0.02; collision box size=0.227 0.133887 0.05
- link r_larm: geometry collision box size=0.135 0.15 0.06; collision cylinder length=0.125 radius=0.045
- link r_lfarm: geometry collision box size=0.13 0.09 0.07; collision cylinder length=0.05 radius=0.03
- link r_lglut: geometry collision box size=0.125 0.05 0.08; collision cylinder length=0.060306 radius=0.02009687
- link r_lleg: geometry collision cylinder length=0.40 radius=0.07; visual mesh filename=package://meshes_unplugged/r_lleg.obj scale=1 1 1
- link r_scap: geometry collision box size=0.02 0.029 0.018; collision box size=0.028 0.090 0.05
- link r_talus: geometry collision cylinder length=0.010059 radius=0.010348; collision cylinder length=0.029542 radius=0.010181
- link r_uarm: geometry collision box size=0.05 0.07 0.15; collision cylinder length=0.11 radius=0.065
- link r_ufarm: geometry collision box size=0.135 0.1 0.045; collision cylinder length=0.125 radius=0.045
- link r_uglut: geometry collision box size=0.05 0.1 0.1; collision cylinder length=0.080842 radius=0.019841
- link r_uleg: geometry collision box size=0.07 0.038 0.14; collision box size=0.07 0.038 0.15
- link utorso: geometry collision box size=0.13 0.50 0.10; collision box size=0.2 0.18 0.10
Joints:
- added joint pelvis_com_fixed: type fixed, parent pelvis, child pelvis_com, origin xyz=0.0111 0 0.0271 rpy=0 -0 0

File: robot_model/atlas/atlas_rel_path.urdf (robot description, URDF)
Before this commit: robot multisense_sl, 33 links, 32 joints
Links:
- added link pelvis_com, mass 0.001
- link head: geometry collision box size=0.0468 0.12 0.1184; collision box size=0.1311 0.12 0.0591
- link l_clav: geometry collision box size=0.1 0.07 0.072; collision cylinder length=0.1525 radius=0.0555
- link l_foot: geometry collision box size=0.1 0.08 0.02; collision box size=0.227 0.133887 0.05
- link l_larm: geometry collision box size=0.135 0.15 0.06; collision cylinder length=0.125 radius=0.045
- link l_lfarm: geometry collision box size=0.13 0.09 0.07; collision cylinder length=0.05 radius=0.03
- link l_lglut: geometry collision box size=0.125 0.05 0.08; collision cylinder length=0.060306 radius=0.02009687
- link l_lleg: geometry collision cylinder length=0.40 radius=0.07; visual mesh filename=meshes_unplugged/l_lleg.obj scale=1 1 1
- link l_scap: geometry collision box size=0.02 0.029 0.018; collision box size=0.028 0.090 0.05
- link l_talus: geometry collision cylinder length=0.010059 radius=0.010348; collision cylinder length=0.029542 radius=0.010181
- link l_uarm: geometry collision box size=0.05 0.07 0.15; collision cylinder length=0.11 radius=0.065
- link l_ufarm: geometry collision box size=0.135 0.1 0.045; collision cylinder length=0.125 radius=0.045
- link l_uglut: geometry collision box size=0.05 0.1 0.1; collision cylinder length=0.080842 radius=0.019841
- link l_uleg: geometry collision box size=0.07 0.038 0.14; collision box size=0.07 0.038 0.15
- link ltorso: geometry visual mesh filename=meshes_unplugged/ltorso.obj scale=1 1 1
- link mtorso: geometry collision cylinder length=0.15 radius=0.02; visual mesh filename=meshes_unplugged/mtorso.obj scale=1 1 1
- link pelvis: geometry collision box size=0.1 0.15 0.2; collision cylinder length=0.05 radius=0.16
- link r_clav: geometry collision box size=0.1 0.07 0.072; collision cylinder length=0.1525 radius=0.0555
- link r_foot: geometry collision box size=0.1 0.08 0.02; collision box size=0.227 0.133887 0.05
- link r_larm: geometry collision box size=0.135 0.15 0.06; collision cylinder length=0.125 radius=0.045
- link r_lfarm: geometry collision box size=0.13 0.09 0.07; collision cylinder length=0.05 radius=0.03
- link r_lglut: geometry collision box size=0.125 0.05 0.08; collision cylinder length=0.060306 radius=0.02009687
- link r_lleg: geometry collision cylinder length=0.40 radius=0.07; visual mesh filename=meshes_unplugged/r_lleg.obj scale=1 1 1
- link r_scap: geometry collision box size=0.02 0.029 0.018; collision box size=0.028 0.090 0.05
- link r_talus: geometry collision cylinder length=0.010059 radius=0.010348; collision cylinder length=0.029542 radius=0.010181
- link r_uarm: geometry collision box size=0.05 0.07 0.15; collision cylinder length=0.11 radius=0.065
- link r_ufarm: geometry collision box size=0.135 0.1 0.045; collision cylinder length=0.125 radius=0.045
- link r_uglut: geometry collision box size=0.05 0.1 0.1; collision cylinder length=0.080842 radius=0.019841
- link r_uleg: geometry collision box size=0.07 0.038 0.14; collision box size=0.07 0.038 0.15
- link utorso: geometry collision box size=0.13 0.50 0.10; collision box size=0.2 0.18 0.10
Joints:
- added joint pelvis_com_fixed: type fixed, parent pelvis, child pelvis_com, origin xyz=0.0111 0 0.0271 rpy=0 -0 0
