Commit message: updated joints, links for dog from atlas

File: robot_model/dog/dog.urdf (robot description, URDF)
Before this commit: robot dog, 13 links, 12 joints
Links:
- added link fl.sole, mass 0.001
- added link fr.sole, mass 0.001
- added link hl.sole, mass 0.001
- added link hr.sole, mass 0.001
- link base: geometry collision mesh filename=package://meshes/base.dae; visual mesh filename=package://meshes/base.dae
- link fl.hip: geometry collision mesh filename=package://meshes/fl.hip.dae; visual mesh filename=package://meshes/fl.hip.dae
- link fl.lleg: geometry collision mesh filename=package://meshes/fl.lleg.dae; visual mesh filename=package://meshes/fl.lleg.dae
- link fl.uleg: geometry collision mesh filename=package://meshes/fl.uleg.dae; visual mesh filename=package://meshes/fl.uleg.dae
- link fr.hip: geometry collision mesh filename=package://meshes/fr.hip.dae; visual mesh filename=package://meshes/fr.hip.dae
- link fr.lleg: geometry collision mesh filename=package://meshes/fr.lleg.dae; visual mesh filename=package://meshes/fr.lleg.dae
- link fr.uleg: geometry collision mesh filename=package://meshes/fr.uleg.dae; visual mesh filename=package://meshes/fr.uleg.dae
- link hl.hip: geometry collision mesh filename=package://meshes/hl.hip.dae; visual mesh filename=package://meshes/hl.hip.dae
- link hl.lleg: geometry collision mesh filename=package://meshes/hl.lleg.dae; visual mesh filename=package://meshes/hl.lleg.dae
- link hl.uleg: geometry collision mesh filename=package://meshes/hl.uleg.dae; visual mesh filename=package://meshes/hl.uleg.dae
- link hr.hip: geometry collision mesh filename=package://meshes/hr.hip.dae; visual mesh filename=package://meshes/hr.hip.dae
- link hr.lleg: geometry collision mesh filename=package://meshes/hr.lleg.dae; visual mesh filename=package://meshes/hr.lleg.dae
- link hr.uleg: geometry collision mesh filename=package://meshes/hr.uleg.dae; visual mesh filename=package://meshes/hr.uleg.dae
Joints:
- added joint fl.sole_fixed: type fixed, parent fl.lleg, child fl.sole, origin xyz=0.023 0 -0.074119 rpy=0 0 0
- added joint fr.sole_fixed: type fixed, parent fr.lleg, child fr.sole, origin xyz=0.023 0 -0.074119 rpy=0 0 0
- added joint hl.sole_fixed: type fixed, parent hl.lleg, child hl.sole, origin xyz=0.023 0 -0.074119 rpy=0 0 0
- added joint hr.sole_fixed: type fixed, parent hr.lleg, child hr.sole, origin xyz=0.023 0 -0.074119 rpy=0 0 0

Commit message: saving rproject repo snapshot

File: robot_model/dog/dog.urdf (robot description, URDF)
Before this commit: robot dog, 17 links, 16 joints
Joints:
- joint fr.hx: origin xyz=0.29785 -0.05500 0.00000 rpy=0 0 0 -> xyz=0.29785 -0.05500 -0.22000 rpy=0 0 0
- joint hr.hx: origin xyz=-0.29785 -0.05500 0.00000 rpy=0 0 0 -> xyz=-0.29785 -0.05500 -0.22000 rpy=0 0 0
